File: electronics/speaking_clock_smd/peripherals.kicad_sch (KiCad schematic)
At the start: 39 parts, among them J2 Conn_01x02_Pin, J3 Conn_01x03_Pin, J4 Conn_01x02_Pin, Q1 IRLML6401, Q2 AO3400A, Q3 AO3400A, SW2 volume_knob, SW3 config, U6 HEF4093B, U7 TPS63070RNMR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

Commit message: take over changes to electronics from test branch
Parts:
- BT1: footprint my_footprints:BatteryHolderCR2032 -> my_footprints:Keytone_CR2032_holder
- D3: footprint LED_SMD:LED_0201_0603Metric -> LED_SMD:LED_0603_1608Metric
- Q1: LCSC (none) -> C382329
- SW3: LCSC C318884 -> (none)
- U9: LCSC (none) -> C910544
Changed lines of the file:
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@@
 			)
 		)
-		(property "Footprint" "my_footprints:BatteryHolderCR2032"
+		(property "Footprint" "my_footprints:Keytone_CR2032_holder"
 			(at 219.964 113.03 90)
 			(effects
@@
 		(property "Description" "Single-cell battery"
 			(at 218.44 113.03 0)
+			(effects
+				(font
+					(size 1.27 1.27)
+				)
+				(hide yes)
+			)
+		)
+		(property "LCSC" ""
+			(at 218.44 113.03 90)
 			(effects
 				(font
@@
 			)
 		)
-		(property "LCSC" "C318884"
+		(property "LCSC" ""
 			(at 116.84 77.47 90)
 			(effects
@@
 			)
 		)
-		(property "Footprint" "LED_SMD:LED_0201_0603Metric"
+		(property "Footprint" "LED_SMD:LED_0603_1608Metric"
 			(at 161.29 147.32 0)
 			(effects
@@
 			)
 		)
+		(property "LCSC" "C382329"
+			(at 34.29 124.46 0)
+			(effects
+				(font
+					(size 1.27 1.27)
+				)
+				(hide yes)
+			)
+		)
 		(pin "1"
 		)
@@
 			(at 232.41 60.96 0)
 			(effects
+				(font
+					(size 1.27 1.27)
+				)
+				(hide yes)
+			)
+		)
+		(property "LCSC" "C910544"
+			(at 232.41 60.96 0)
+			(effects
