File: electronics/speaking_clock_smd/speaking_clock_smd.kicad_pcb (KiCad board)
At the start: 4 copper layers, 60 x 79 mm, 86 parts, among them J1 USB_C_Receptacle_USB2.0, J2 Conn_01x02_Pin, J3 Conn_01x03_Pin, J4 Conn_01x02_Pin, Q1 IRLML6401, Q2 AO3400A, Q3 AO3400A, SW1 reset, SW2 volume_knob, SW3 config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

Commit message: take over changes to electronics from test branch
Parts:
- added U20: ~, my_footprints:JLC_tooling_hole, F.Cu at (18.0, -45.0)
- added U21: ~, my_footprints:JLC_tooling_hole, F.Cu at (-27.0, 8.00)
- added U22: ~, my_footprints:JLC_tooling_hole, F.Cu at (18.0, 21.0)
- BT1: footprint my_footprints:BatteryHolderCR2032 -> my_footprints:Keytone_CR2032_holder
- D3: footprint LED_SMD:LED_0201_0603Metric -> LED_SMD:LED_0603_1608Metric
- moved R22 2.86 mm to (9.47, -8.94)
- moved R26 1.19 mm to (26.0, 12.4)
- turned BT1 to 0 degrees
Routing:
- net VBat: track 90.6 -> 96.6 mm
- net GND: track 87.2 -> 82.6 mm, vias 173 -> 224
- net ON: track 39.5 -> 42.2 mm
- net Net-(D3-A): track 1.67 -> 3.09 mm
- net +3.3V: track 183.1 -> 182.2 mm
- net Net-(BT1-+): track 60.9 -> 61.1 mm, vias 2 -> 1
